File: ATF15xxProgBoard/ATF15xxProgBoard.kicad_pcb (KiCad board)
At the start: 4 copper layers, 71.1 x 96.2 mm, 20 parts, among them J1 Conn_02x05_Odd_Even, J2 Conn_02x07_Odd_Even, J3 USB_C_Receptacle_PowerOnly_6P, J4 Conn_01x02_Pin, J5 Jack-DC, J6 Conn_02x16_Counter_Clockwise, J7 Conn_02x16_Counter_Clockwise, J8 Conn_02x03_Odd_Even

Commit message: COMMERCIAL: Full redesign as programmer
Parts:
- removed J3: USB_C_Receptacle_PowerOnly_6P, Connector_USB:USB_C_Receptacle_Palconn_UTC16-G
- removed J4: Conn_01x02_Pin, Connector_PinHeader_2.54mm:PinHeader_1x03_P2.54mm_Vertical
- removed J5: Jack-DC, Connector_BarrelJack:BarrelJack_Horizontal
- removed R2: 5.1K, Resistor_THT:R_Axial_DIN0207_L6.3mm_D2.5mm_P10.16mm_Horizontal
- added C10: 4.7u, Capacitor_SMD:C_0603_1608Metric, F.Cu at (169.9, 123.0)
- added C11: 4.7u, Capacitor_SMD:C_0603_1608Metric, F.Cu at (171.7, 123.0)
- added C6: 10u, Capacitor_SMD:C_0805_2012Metric_Pad1.18x1.45mm_HandSolder, F.Cu at (171.0, 104.7)
- added C7: 22p, Capacitor_SMD:C_0603_1608Metric_Pad1.08x0.95mm_HandSolder, F.Cu at (160.0, 127.2)
- added C8: 22p, Capacitor_SMD:C_0603_1608Metric_Pad1.08x0.95mm_HandSolder, F.Cu at (148.6, 126.6)
- added C9: 1u, Capacitor_SMD:C_0805_2012Metric_Pad1.18x1.45mm_HandSolder, F.Cu at (148.8, 102.6)
- added D1: 1N4148, Diode_SMD:D_SOD-123, F.Cu at (165.9, 90.8)
- added J10: Conn_02x03_Odd_Even, Connector_PinHeader_2.54mm:PinHeader_2x03_P2.54mm_Vertical, F.Cu at (161.8, 122.9)
- added J9: USB_C, Connector_USB:USB_C_Receptacle_Palconn_UTC16-G, F.Cu at (170.9, 111.2)
- added JP2: Voltage, Connector_PinHeader_2.54mm:PinHeader_1x03_P2.54mm_Vertical, F.Cu at (164.7, 126.6)
- added L1: 4.7uH, Inductor_SMD:L_0805_2012Metric_Pad1.05x1.20mm_HandSolder, F.Cu at (165.8, 98.8)
- added LED2: GREEN, LED_SMD:LED_0603_1608Metric_Pad1.05x0.95mm_HandSolder, F.Cu at (166.0, 64.7)
- added LED3: ORANGE, LED_SMD:LED_0603_1608Metric_Pad1.05x0.95mm_HandSolder, F.Cu at (170.6, 64.7)
- added R10: 100K, Resistor_SMD:R_0603_1608Metric, F.Cu at (161.2, 96.1)
- added R11: 10K, Resistor_SMD:R_0603_1608Metric, F.Cu at (161.2, 97.8)
- added R12: 2.2K, Resistor_SMD:R_0603_1608Metric, F.Cu at (170.2, 90.8)
- added R4: 5.1K, Resistor_SMD:R_0603_1608Metric_Pad0.98x0.95mm_HandSolder, F.Cu at (164.6, 105.1)
- added R5: 5.1K, Resistor_SMD:R_0603_1608Metric_Pad0.98x0.95mm_HandSolder, F.Cu at (164.6, 116.6)
- added R6: 22R, Resistor_SMD:R_0603_1608Metric_Pad0.98x0.95mm_HandSolder, F.Cu at (163.8, 109.9)
- added R7: 22R, Resistor_SMD:R_0603_1608Metric_Pad0.98x0.95mm_HandSolder, F.Cu at (163.8, 112.6)
- added R8: 10k, Resistor_SMD:R_0603_1608Metric_Pad0.98x0.95mm_HandSolder, F.Cu at (160.8, 107.5)
- added R9: 2K, Resistor_SMD:R_0603_1608Metric, F.Cu at (170.6, 66.4)
- added U3: ATmega32U4-AU, Package_QFP:TQFP-44_10x10mm_P0.8mm, F.Cu at (153.2, 115.4)
- added U4: MT3540, Package_TO_SOT_SMD:SOT-23-5, F.Cu at (165.9, 95.2)
- added U5: AP2127K-3.3, Package_TO_SOT_SMD:SOT-23-5, F.Cu at (171.2, 119.6)
- added Y1: 8MHz, Crystal:Crystal_SMD_5032-2Pin_5.0x3.2mm_HandSoldering, F.Cu at (154.5, 126.6)
- C1: value 470u -> 10u; footprint Capacitor_THT:CP_Radial_D10.0mm_P3.80mm -> Capacitor_SMD:C_0805_2012Metric_Pad1.18x1.45mm_HandSolder
- C2: value 100n -> 10u; footprint Capacitor_THT:C_Rect_L4.0mm_W2.5mm_P2.50mm -> Capacitor_SMD:C_0805_2012Metric_Pad1.18x1.45mm_HandSolder
- C3, C4, C5: footprint Capacitor_THT:C_Rect_L4.0mm_W2.5mm_P2.50mm -> Capacitor_SMD:C_0603_1608Metric_Pad1.08x0.95mm_HandSolder
- LED1: footprint LED_THT:LED_D5.0mm -> LED_SMD:LED_0603_1608Metric_Pad1.05x0.95mm_HandSolder
- R1: value 1K -> 2K; footprint Resistor_THT:R_Axial_DIN0207_L6.3mm_D2.5mm_P10.16mm_Horizontal -> Resistor_SMD:R_0603_1608Metric
- R3: value 5.1K -> 2K; footprint Resistor_THT:R_Axial_DIN0207_L6.3mm_D2.5mm_P10.16mm_Horizontal -> Resistor_SMD:R_0603_1608Metric
- moved R3 39.1 mm to (165.9, 66.4), turned to 180 degrees
- moved C1 30.0 mm to (169.2, 95.3), turned to -90 degrees
- moved C3 8.53 mm to (161.9, 84.1), turned to 90 degrees
- moved LED1 6.69 mm to (161.1, 64.7)
- moved C2 5.37 mm to (161.4, 92.9)
- moved R1 3.54 mm to (161.1, 66.4), turned to 0 degrees
- moved C5 2.64 mm to (155.1, 106.7), turned to 180 degrees
Connections:
- net IO1 renamed /IO1
- net IO10 renamed /IO10
- net IO11 renamed /IO11
- net IO12 renamed /IO12
- net IO13 renamed /IO13
- net IO14 renamed /IO14
- net IO15 renamed /IO15
- net IO16 renamed /IO16
- net IO17 renamed /IO17
- net IO18 renamed /IO18
- net IO19 renamed /IO19
- net IO2 renamed /IO2
- net IO20 renamed /IO20
- net IO21 renamed /IO21
- net IO22 renamed /IO22
- net IO23 renamed /IO23
- net IO25 renamed /IO25
- net IO26 renamed /IO26
- net IO27 renamed /IO27
- net IO28 renamed /IO28
- net IO3 renamed /IO3
- net IO30 renamed /IO30
- net IO31 renamed /IO31
- net IO32 renamed /IO32
- net IO33 renamed /IO33
- net IO34 renamed /IO34
- net IO35 renamed /IO35
- net IO36 renamed /IO36
- net IO37 renamed /IO37
- net IO38 renamed /IO38
- net IO39 renamed /IO39
- net IO40 renamed /IO40
- net IO41 renamed /IO41
- net IO42 renamed /IO42
- net IO43 renamed /IO43
- net IO44 renamed /IO44
- net IO45 renamed /IO45
- net IO46 renamed /IO46
- net IO47 renamed /IO47
- net IO48 renamed /IO48
- net IO49 renamed /IO49
- net IO5 renamed /IO5
- net IO50 renamed /IO50
- net IO52 renamed /IO52
- net IO53 renamed /IO53
- net IO54 renamed /IO54
- net IO55 renamed /IO55
- net IO56 renamed /IO56
- net IO57 renamed /IO57
- net IO58 renamed /IO58
- net IO6 renamed /IO6
- net IO60 renamed /IO60
- net IO61 renamed /IO61
- net IO62 renamed /IO62
- net IO63 renamed /IO63
- net IO64 renamed /IO64
- net IO65 renamed /IO65
- net IO66 renamed /IO66
- net IO7 renamed /IO7
- net IO8 renamed /IO8
- C2 pad 1: VCC -> Net-(D1-K)
- JP1 pad 1: VCC -> unconnected-(JP1-A-Pad1)
- R3 pad 1: GND -> VCC
Routing:
- net OE1/I: track 103.0 -> 212.6 mm, vias 2 -> 4
- net GND: track 176.1 -> 250.6 mm, vias 0 -> 17
- net VCC: track 130.5 -> 204.4 mm, vias 2 -> 15
- net /~{RDY}: track 0.00 -> 61.4 mm, vias 0 -> 2
- net TDI: track 97.8 -> 158.7 mm, vias 1 -> 2
- net /~{ACT}: track 0.00 -> 60.1 mm, vias 0 -> 2
- net VBUS: track 0.00 -> 56.3 mm, vias 0 -> 5
- net TMS: track 93.7 -> 143.5 mm, vias 0 -> 1
- net TCK: track 145.2 -> 181.8 mm, vias 1 -> 3
- net /~{RESET}: track 0.00 -> 27.5 mm, vias 0 -> 1
- net /VPP_EN: track 0.00 -> 24.9 mm, vias 0 -> 2
- net /PDI: track 0.00 -> 24.5 mm, vias 0 -> 1
- net +3V3: track 0.00 -> 21.7 mm, vias 0 -> 1
- net Net-(U3-UCAP): track 0.00 -> 19.9 mm, vias 0 -> 2
- net /SCLK: track 0.00 -> 19.5 mm, vias 0 -> 1
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Other:
- board text added: "(!)️ OE/I"
- board text added: "3.3V"
- board text added: "5V"
- board text added: "@roscopeco"
- board text added: "ACT"
- board text added: "ATF1504 or ATF1508"
- board text added: "GCLK1"
- board text added: "GCLK2"
- board text added: "GCLK3"
- board text added: "GCLR"
- board text added: "READY"
- board text removed: "2"
- board text removed: "43"
- board text removed: "81"
- board text removed: "83"
- board text removed: "84"
- board text removed: ":44P"
- board text removed: ":84P"
- board text removed: "@roscopeco 2024"
- board text removed: "ATF1504"
- board text removed: "CENTER POSITIVE"

Commit message: Minor tidy up
Routing:
- net /IO1: track 125.8 -> 131.1 mm
- net /IO8: track 96.3 -> 99.7 mm
- net /IO7: track 117.9 -> 121.0 mm
- net /IO13: track 117.4 -> 119.3 mm
- net /IO5: track 145.2 -> 143.5 mm
- net GND: track 250.6 -> 251.7 mm
- net /IO33: track 49.8 -> 50.9 mm
- net /IO40: track 60.3 -> 61.1 mm
- net /IO23: track 81.2 -> 80.5 mm
- net /PDO: track 16.7 -> 16.1 mm
- net /IO35: track 49.8 -> 50.4 mm
- net VCC: track 204.4 -> 203.8 mm
- net /IO14: track 79.8 -> 79.2 mm
- net /32_XTAL1: track 11.1 -> 10.5 mm
- net /IO34: track 49.6 -> 50.2 mm
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
Commit message: Open sourcing
Connections:
- JP1 pad 1: unconnected-(JP1-A-Pad1) -> VCC
Routing:
- net /IO12: track 95.5 -> 96.6 mm
- net TDI: track 158.3 -> 159.3 mm
- net /IO2: track 154.7 -> 155.5 mm
- net /IO10: track 103.2 -> 103.9 mm
- net Net-(J1-Pin_4): track 37.2 -> 36.7 mm
