File: ATF15xxProgBoard/ATF15xxProgBoard.kicad_sch (KiCad schematic)
At the start: 43 parts, among them J1 Conn_02x05_Odd_Even, J1 USB_C, J2 Conn_02x03_Odd_Even, J2 Conn_02x07_Odd_Even, J6 Conn_02x16_Counter_Clockwise, J7 Conn_02x16_Counter_Clockwise, J8 Conn_02x03_Odd_Even, U1 ATmega32U4-AU, U4 MT3540, U6 AP2127K-3.3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

Commit message: Open sourcing
Connections:
- net VCC: now also JP1.1 (A)
Other:
- moved on the sheet: JP1
